File: board/board.kicad_pcb (KiCad board)
At the start: 2 copper layers, 21 x 13 mm, 1 part

Commit message: initial b149
Parts:
- added C1: 100nF, Capacitor_SMD:C_0402_1005Metric, B.Cu at (65.1, 83.6)
- added C10: 100nF, Capacitor_SMD:C_0402_1005Metric, B.Cu at (68.0, 76.3)
- added C11: 100nF, Capacitor_SMD:C_0402_1005Metric, B.Cu at (76.2, 68.2)
- added C12: 100nF, Capacitor_SMD:C_0402_1005Metric, B.Cu at (83.9, 71.7)
- added C13: 100nF, Capacitor_SMD:C_0402_1005Metric, B.Cu at (88.2, 76.4)
- added C14: 100nF, Capacitor_SMD:C_0402_1005Metric, B.Cu at (85.3, 73.2)
- added C15: 100nF, Capacitor_SMD:C_0402_1005Metric, B.Cu at (86.3, 85.5)
- added C16: 100nF, Capacitor_SMD:C_0402_1005Metric, B.Cu at (84.3, 87.5)
- added C17: 100nF, Capacitor_SMD:C_0402_1005Metric, B.Cu at (83.7, 88.2)
- added C18: 100nF, Capacitor_SMD:C_0402_1005Metric, B.Cu at (81.9, 89.8)
- added C19: 100nF, Capacitor_SMD:C_0402_1005Metric, B.Cu at (72.8, 88.9)
- added C2: 10uF, Capacitor_SMD:C_0603_1608Metric, B.Cu at (65.6, 84.8)
- added C20: 100nF, Capacitor_SMD:C_0402_1005Metric, B.Cu at (85.7, 86.2)
- added C21: 100nF, Capacitor_SMD:C_0402_1005Metric, B.Cu at (85.0, 86.8)
- added C22: 100nF, Capacitor_SMD:C_0402_1005Metric, B.Cu at (87.9, 84.0)
- added C23: 100nF, Capacitor_SMD:C_0402_1005Metric, B.Cu at (75.4, 91.6)
- added C24: 100nF, Capacitor_SMD:C_0402_1005Metric, B.Cu at (74.2, 90.3)
- added C25: 12pF, Capacitor_SMD:C_0402_1005Metric, B.Cu at (70.4, 67.0)
- added C26: 12pF, Capacitor_SMD:C_0402_1005Metric, B.Cu at (68.5, 67.0)
- added C27: 100nF, Capacitor_SMD:C_0402_1005Metric, B.Cu at (69.0, 84.7)
- added C3: 100nF, Capacitor_SMD:C_0402_1005Metric, B.Cu at (66.1, 76.3)
- added C4: 10uF, Capacitor_SMD:C_0603_1608Metric, B.Cu at (65.5, 77.5)
- added C5: 100nF, Capacitor_SMD:C_0402_1005Metric, B.Cu at (74.1, 69.6)
- added C6: 100nF, Capacitor_SMD:C_0402_1005Metric, B.Cu at (86.0, 73.9)
- added C7: 100nF, Capacitor_SMD:C_0402_1005Metric, B.Cu at (82.0, 70.2)
- added C8: 100nF, Capacitor_SMD:C_0402_1005Metric, B.Cu at (89.7, 79.2)
- added C9: 100nF, Capacitor_SMD:C_0402_1005Metric, B.Cu at (71.0, 72.9)
- added J1: 020_1000BASE-T_with_CT, on_edge:on_edge_2x10_host, F.Cu at (101.0, 26.5)
- added J2: 020_1000BASE-T_with_CT, on_edge:on_edge_2x10_host, F.Cu at (101.0, 58.5)
- added J3: 020_1000BASE-T_with_CT, on_edge:on_edge_2x10_host, F.Cu at (101.0, 90.5)
- added J4: 020_1000BASE-T_with_CT, on_edge:on_edge_2x10_host, F.Cu at (101.0, 122.5)
- added J5: 020_1000BASE-T_with_CT, on_edge:on_edge_2x10_host, F.Cu at (101.0, 154.5)
- added J6: 011_GPIO, on_edge:on_edge_2x05_device, F.Cu at (56.0, 26.5)
- added L1: 2.2uH, Inductor_SMD:L_Sunlord_MWSA0402S, B.Cu at (64.2, 80.7)
- added R1: 1k, Resistor_SMD:R_0402_1005Metric, B.Cu at (67.7, 84.6)
- added R10: 2.49k, Resistor_SMD:R_0402_1005Metric, B.Cu at (90.2, 81.4)
- added R2: 4.7k, Resistor_SMD:R_0402_1005Metric, B.Cu at (67.9, 75.3)
- added R3: 4.7k, Resistor_SMD:R_0402_1005Metric, B.Cu at (67.9, 74.4)
- added R4: 4.7k, Resistor_SMD:R_0402_1005Metric, B.Cu at (67.9, 73.5)
- added R5: 4.7k, Resistor_SMD:R_0402_1005Metric, B.Cu at (67.9, 72.5)
- added R6: 4.7k, Resistor_SMD:R_0402_1005Metric, B.Cu at (67.9, 71.5)
- added R7: 4.7k, Resistor_SMD:R_0402_1005Metric, B.Cu at (73.1, 67.7)
- added R8: 4.7k, Resistor_SMD:R_0402_1005Metric, B.Cu at (73.1, 69.6)
- added R9: 4.7k, Resistor_SMD:R_0402_1005Metric, B.Cu at (72.1, 69.6)
- added U1: RTL8367S-CG, Package_QFP:LQFP-128_14x14mm_P0.4mm, B.Cu at (78.0, 80.0)
- added Y1: 25MhZ, Crystal:Crystal_SMD_3225-4Pin_3.2x2.5mm, B.Cu at (69.5, 69.3)
- moved LOGO1 102.6 mm to (64.0, 43.0)
Routing:
- net GND: track 0.00 -> 379.7 mm, vias 0 -> 44
- net /3.3V: track 0.00 -> 304.1 mm, vias 0 -> 18
- net /5V: track 0.00 -> 187.3 mm, vias 0 -> 5
- net /switch/1V: track 0.00 -> 95.4 mm, vias 0 -> 12
- net /switch/P4D-: track 0.00 -> 90.6 mm, vias 0 -> 1
- net /switch/P4D+: track 0.00 -> 89.8 mm, vias 0 -> 1
- net /switch/P4C-: track 0.00 -> 87.7 mm, vias 0 -> 1
- net /switch/P4C+: track 0.00 -> 87.7 mm, vias 0 -> 1
- net /switch/P4B-: track 0.00 -> 83.3 mm, vias 0 -> 1
- net /switch/P4B+: track 0.00 -> 82.8 mm, vias 0 -> 1
- net /switch/P4A-: track 0.00 -> 79.3 mm, vias 0 -> 1
- net /switch/P4A+: track 0.00 -> 79.1 mm, vias 0 -> 1
- net /switch/P3D-: track 0.00 -> 60.9 mm, vias 0 -> 1
- net /switch/P3D+: track 0.00 -> 60.2 mm, vias 0 -> 1
- net /switch/P0A+: track 0.00 -> 60.2 mm, vias 0 -> 1
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Other:
- board size 21 x 13 mm -> 45 x 157 mm
- copper layers 2 -> 4
- board text added: "osf.b149.V1.0"
