File: board/switch.kicad_sch (KiCad schematic)
At the start: 40 parts, among them U1 RTL8367S-CG, Y1 25MhZ

Commit message: added lcsc part numbers
Parts:
- C1, C10, C11, C12, C13, C14, C15, C16, C17, C18, C19, C20, C21, C22, C23, C24, C27, C3, C5, C6, C7, C8, C9: lcsc (none) -> C1525
- C2, C4: lcsc (none) -> C19702
- C25, C26: lcsc (none) -> C1547
- L1: lcsc (none) -> C408335
- R1: lcsc (none) -> C11702
- R10: lcsc (none) -> C25884
- R2, R3, R4, R5, R6, R7, R8, R9: lcsc (none) -> C25900
- U1: lcsc (none) -> C2760849
- Y1: lcsc (none) -> C9006
Changed lines of the file:
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@@
+      (effects (font (size 1.27 1.27)) hide)
+    )
+    (property "lcsc" "C1525" (at 243.205 91.44 0)
       (effects (font (size 1.27 1.27)) hide)
     )
@@
       (effects (font (size 1.27 1.27)) hide)
     )
+    (property "lcsc" "C1525" (at 255.27 91.44 0)
+      (effects (font (size 1.27 1.27)) hide)
+    )
     (pin "1")
     (pin "2")
@@
       (effects (font (size 1.27 1.27)) hide)
     )
+    (property "lcsc" "C25900" (at 133.35 36.195 0)
+      (effects (font (size 1.27 1.27)) hide)
+    )
     (pin "1")
     (pin "2")
@@
       (effects (font (size 1.27 1.27)) hide)
     )
+    (property "lcsc" "C1525" (at 231.14 133.35 0)
+      (effects (font (size 1.27 1.27)) hide)
+    )
     (pin "1")
     (pin "2")
@@
       (effects (font (size 1.27 1.27)) hide)
     )
+    (property "lcsc" "C1525" (at 243.205 119.38 0)
+      (effects (font (size 1.27 1.27)) hide)
+    )
     (pin "1")
     (pin "2")
@@
       (effects (font (size 1.27 1.27)) hide)
     )
+    (property "lcsc" "C25900" (at 140.97 26.67 0)
+      (effects (font (size 1.27 1.27)) hide)
+    )
     (pin "1")
     (pin "2")
@@
       (effects (font (size 1.27 1.27)) hide)
     )
+    (property "lcsc" "C1525" (at 255.27 119.38 0)
+      (effects (font (size 1.27 1.27)) hide)
+    )
     (pin "1")
     (pin "2")
@@
       (effects (font (size 1.27 1.27)) hide)
     )
+    (property "lcsc" "C1525" (at 219.075 105.41 0)
+      (effects (font (size 1.27 1.27)) hide)
+    )
     (pin "1")
     (pin "2")
@@
       (effects (font (size 1.27 1.27)) hide)
     )
+    (property "lcsc" "C19702" (at 187.96 40.64 0)
+      (effects (font (size 1.27 1.27)) hide)
+    )
     (pin "1")
     (pin "2")
@@
     )
     (property "Datasheet" "~" (at 219.075 119.38 0)
+      (effects (font (size 1.27 1.27)) hide)
+    )
+    (property "lcsc" "C1525" (at 219.075 119.38 0)
       (effects (font (size 1.27 1.27)) hide)
     )
@@
       (effects (font (size 1.27 1.27)) hide)
     )
+    (property "lcsc" "C25900" (at 115.57 21.59 0)
+      (effects (font (size 1.27 1.27)) hide)
+    )
     (pin "1")
     (pin "2")
@@
       (effects (font (size 1.27 1.27)) hide)
     )
+    (property "lcsc" "C1525" (at 205.74 105.41 0)
+      (effects (font (size 1.27 1.27)) hide)
+    )
     (pin "1")
     (pin "2")
@@
     )
     (property "Datasheet" "~" (at 267.335 104.775 0)
+      (effects (font (size 1.27 1.27)) hide)
+    )
+    (property "lcsc" "C1525" (at 267.335 104.775 0)
       (effects (font (size 1.27 1.27)) hide)
     )
@@
       (effects (font (size 1.27 1.27)) hide)
     )
+    (property "lcsc" "C25900" (at 115.57 36.83 0)
+      (effects (font (size 1.27 1.27)) hide)
+    )
     (pin "1")
     (pin "2")
@@
       (effects (font (size 1.27 1.27)) hide)
     )
+    (property "lcsc" "C1525" (at 243.205 105.41 0)
+      (effects (font (size 1.27 1.27)) hide)
+    )
     (pin "1")
     (pin "2")
@@
       (effects (font (size 1.27 1.27)) hide)
     )
+    (property "lcsc" "C1525" (at 176.53 40.64 0)
+      (effects (font (size 1.27 1.27)) hide)
+    )
     (pin "1")
     (pin "2")
@@
     )
     (property "Datasheet" "~" (at 143.51 31.75 0)
+      (effects (font (size 1.27 1.27)) hide)
+    )
+    (property "lcsc" "C25900" (at 143.51 31.75 0)
       (effects (font (size 1.27 1.27)) hide)
     )
@@
       (effects (font (size 1.27 1.27)) hide)
     )
+    (property "lcsc" "C11702" (at 180.34 66.04 0)
+      (effects (font (size 1.27 1.27)) hide)
+    )
     (pin "1")
     (pin "2")
@@
     )
     (property "Datasheet" "~" (at 231.14 105.41 0)
+      (effects (font (size 1.27 1.27)) hide)
+    )
+    (property "lcsc" "C1525" (at 231.14 105.41 0)
       (effects (font (size 1.27 1.27)) hide)
     )
@@
       (effects (font (size 1.27 1.27)) hide)
     )
+    (property "lcsc" "C408335" (at 191.77 55.88 0)
+      (effects (font (size 1.27 1.27)) hide)
+    )
     (pin "2")
     (pin "1")
@@
       (effects (font (size 1.27 1.27)) hide)
     )
+    (property "lcsc" "C1525" (at 231.14 91.44 0)
+      (effects (font (size 1.27 1.27)) hide)
+    )
     (pin "1")
     (pin "2")
@@
       (effects (font (size 1.27 1.27)) hide)
     )
+    (property "lcsc" "C1525" (at 231.14 119.38 0)
+      (effects (font (size 1.27 1.27)) hide)
+    )
     (pin "1")
     (pin "2")
@@
       (effects (font (size 1.27 1.27)) hide)
     )
+    (property "lcsc" "C25900" (at 146.05 36.195 0)
+      (effects (font (size 1.27 1.27)) hide)
+    )
     (pin "1")
     (pin "2")
@@
     )
     (property "Datasheet" "~" (at 205.74 91.44 0)
+      (effects (font (size 1.27 1.27)) hide)
+    )
+    (property "lcsc" "C1525" (at 205.74 91.44 0)
       (effects (font (size 1.27 1.27)) hide)
     )
@@
       (effects (font (size 1.27 1.27)) hide)
     )
+    (property "lcsc" "C25884" (at 120.65 166.37 0)
+      (effects (font (size 1.27 1.27)) hide)
+    )
     (pin "1")
     (pin "2")
@@
     )
     (property "Datasheet" "~" (at 128.27 31.115 0)
+      (effects (font (size 1.27 1.27)) hide)
+    )
+    (property "lcsc" "C25900" (at 128.27 31.115 0)
       (effects (font (size 1.27 1.27)) hide)
     )
@@
     )
     (property "Datasheet" "" (at 90.17 149.86 90)
+      (effects (font (size 1.27 1.27)) hide)
+    )
+    (property "lcsc" "C2760849" (at 72.39 52.07 0)
       (effects (font (size 1.27 1.27)) hide)
     )
@@
       (effects (font (size 1.27 1.27)) hide)
     )
+    (property "lcsc" "C1525" (at 219.075 133.35 0)
+      (effects (font (size 1.27 1.27)) hide)
+    )
     (pin "1")
     (pin "2")
@@
       (effects (font (size 1.27 1.27)) hide)
     )
+    (property "lcsc" "C1525" (at 200.66 60.96 0)
+      (effects (font (size 1.27 1.27)) hide)
+    )
     (pin "1")
     (pin "2")
@@
       (effects (font (size 1.27 1.27)) hide)
     )
+    (property "lcsc" "C1547" (at 125.095 24.13 0)
+      (effects (font (size 1.27 1.27)) hide)
+    )
     (pin "1")
     (pin "2")
@@
       (effects (font (size 1.27 1.27)) hide)
     )
+    (property "lcsc" "C1525" (at 205.74 119.38 0)
+      (effects (font (size 1.27 1.27)) hide)
+    )
     (pin "1")
     (pin "2")
@@
       (effects (font (size 1.27 1.27)) hide)
     )
+    (property "lcsc" "C1525" (at 255.27 105.41 0)
+      (effects (font (size 1.27 1.27)) hide)
+    )
     (pin "1")
     (pin "2")
@@
       (effects (font (size 1.27 1.27)) hide)
     )
+    (property "lcsc" "C1525" (at 205.74 133.35 0)
+      (effects (font (size 1.27 1.27)) hide)
+    )
     (pin "1")
     (pin "2")
@@
       (effects (font (size 1.27 1.27)) hide)
     )
+    (property "lcsc" "C1525" (at 219.075 91.44 0)
+      (effects (font (size 1.27 1.27)) hide)
+    )
     (pin "1")
     (pin "2")
@@
     )
     (property "Datasheet" "~" (at 255.27 133.35 0)
+      (effects (font (size 1.27 1.27)) hide)
+    )
+    (property "lcsc" "C1525" (at 255.27 133.35 0)
       (effects (font (size 1.27 1.27)) hide)
     )
@@
       (effects (font (size 1.27 1.27)) hide)
     )
+    (property "lcsc" "C9006" (at 121.92 31.115 0)
+      (effects (font (size 1.27 1.27)) hide)
+    )
     (pin "1")
     (pin "4")
@@
     )
     (property "Datasheet" "~" (at 243.205 133.35 0)
+      (effects (font (size 1.27 1.27)) hide)
+    )
+    (property "lcsc" "C1525" (at 243.205 133.35 0)
       (effects (font (size 1.27 1.27)) hide)
     )
@@
       (effects (font (size 1.27 1.27)) hide)
     )
+    (property "lcsc" "C1547" (at 118.745 24.13 0)
+      (effects (font (size 1.27 1.27)) hide)
+    )
     (pin "1")
     (pin "2")
@@
       (effects (font (size 1.27 1.27)) hide)
     )
+    (property "lcsc" "C25900" (at 113.03 18.415 0)
+      (effects (font (size 1.27 1.27)) hide)
+    )
     (pin "1")
     (pin "2")
@@
       (effects (font (size 1.27 1.27)) hide)
     )
+    (property "lcsc" "C19702" (at 212.09 60.96 0)
+      (effects (font (size 1.27 1.27)) hide)
+    )
